Commit message: Test Operation
modify 03-origins.urdf

File: urdf/03-origins.urdf (robot description, URDF)
Before this commit: robot origins, 2 links, 1 joints
Joints:
- joint base_to_right_leg: axis (none) -> 0 1 0; limit (none) -> lower=-1.5702 upper=1.5702 effort=1000 velocity=0.5; type fixed -> revolute
